Commit message: modified:   .gitignore 	modified:   README.md 	modified:   mower_ws/src/mower_bringup/launch/bringup_pico.launch.py 	deleted:    mower_ws/src/mower_bringup/launch/bringup_real.launch.py 	modified:   mower_ws/src/mower_description/urdf/mower.urdf.xacro 	modified:   mower_ws/src/pico_control_hardware/CMakeLists.txt 	modified:   mower_ws/src/pico_control_hardware/package.xml 	mower_ws/src/mower_bringup/config/coverage_params.yaml 	mower_ws/src/mower_bringup/config/nav2_params.yaml 	mower_ws/src/mower_bringup/config/twist_mux.yaml 	mower_ws/src/mower_bringup/launch/__pycache__/bringup_pico_rtab.launch.cpython-312.pyc 	mower_ws/src/mower_bringup/launch/bringup_pico_rtab.launch.py 	mower_ws/src/mower_bringup/launch/foxglove_bridge.launch.py 	mower_ws/src/mower_bringup/launch/nav2.launch.py 	mower_ws/src/mower_bringup/launch/opennav_coverage.launch.py 	mower_ws/src/mower_bringup/launch/rtabmap.launch.py 	mower_ws/src/mower_bringup/scripts/ 	mower_ws/src/mower_description/urdf/mower.urdf.xacro.orig

File: mower_ws/src/mower_description/urdf/mower.urdf.xacro (robot description, xacro)
@@ -12,4 +12,9 @@
   <xacro:property name="front_wheel_radius" value="0.045"/>
   <xacro:property name="front_wheel_offset" value="0.05"/>
+  <!-- mower blades (piatti di taglio) -->
+  <xacro:property name="blade_radius" value="0.11"/>
+  <xacro:property name="blade_thickness" value="0.003"/>
+  <xacro:property name="blade_offset_y" value="0.11"/>
+  <xacro:property name="blade_offset_x" value="0.0"/>
   <!-- sim toggle -->
   <xacro:property name="use_sim" value="false"/>
@@ -547,3 +552,55 @@
   </gazebo>
   </xacro:if>
+  <!-- Cutting Blades (two discs under chassis) [moved to end] -->
+  <joint name="blade_left_joint" type="fixed">
+    <parent link="chassis"/>
+    <!-- Place at bottom of chassis: z = -(base_height/2 + blade_thickness/2) -->
+    <child link="blade_left"/>
+    <origin xyz="${blade_offset_x} ${blade_offset_y} -${base_height/2.0 + blade_thickness/2.0}" rpy="0 0 0"/>
+  </joint>
+  <link name="blade_left">
+    <visual>
+      <origin xyz="0 0 0" rpy="0 0 0"/>
+      <geometry>
+        <cylinder radius="${blade_radius}" length="${blade_thickness}"/>
+      </geometry>
+      <material name="blade_mat"><color rgba="0.6 0.6 0.6 1.0"/></material>
+    </visual>
+    <collision>
+      <origin xyz="0 0 0" rpy="0 0 0"/>
+      <geometry>
+        <cylinder radius="${blade_radius}" length="${blade_thickness}"/>
+      </geometry>
+    </collision>
+    <inertial>
+      <mass value="0.2"/>
+      <origin xyz="0 0 0" rpy="0 0 0"/>
+      <inertia ixx="1e-4" iyy="1e-4" izz="1e-4" ixy="0" ixz="0" iyz="0"/>
+    </inertial>
+  </link>
+  <joint name="blade_right_joint" type="fixed">
+    <parent link="chassis"/>
+    <child link="blade_right"/>
+    <origin xyz="${blade_offset_x} -${blade_offset_y} -${base_height/2.0 + blade_thickness/2.0}" rpy="0 0 0"/>
+  </joint>
+  <link name="blade_right">
+    <visual>
+      <origin xyz="0 0 0" rpy="0 0 0"/>
+      <geometry>
+        <cylinder radius="${blade_radius}" length="${blade_thickness}"/>
+      </geometry>
+      <material name="blade_mat"/>
+    </visual>
+    <collision>
+      <origin xyz="0 0 0" rpy="0 0 0"/>
+      <geometry>
+        <cylinder radius="${blade_radius}" length="${blade_thickness}"/>
+      </geometry>
+    </collision>
+    <inertial>
+      <mass value="0.2"/>
+      <origin xyz="0 0 0" rpy="0 0 0"/>
+      <inertia ixx="1e-4" iyy="1e-4" izz="1e-4" ixy="0" ixz="0" iyz="0"/>
+    </inertial>
+  </link>
 </robot>

Commit message: feat: aumenta il baudrate seriale a 230400 e rimuove il package di simulazione

File: mower_ws/src/mower_description/urdf/mower.urdf.xacro (robot description, xacro)
@@ -21,5 +21,5 @@
   <!-- ros2_control -->
   <xacro:property name="port" value="/dev/ttyAMA0"/>
-  <xacro:property name="baud" value="115200"/>
+  <xacro:property name="baud" value="230400"/>
   <ros2_control name="MowerHardware" type="system">
     <hardware>

Commit message: Update mower.urdf.xacro
Update mower.urdf.xacro

File: mower_ws/src/mower_description/urdf/mower.urdf.xacro (robot description, xacro)
@@ -3,13 +3,13 @@
   <!-- Parameters -->
   <xacro:property name="wheel_radius" value="0.15"/>
-  <xacro:property name="wheel_width" value="0.06"/>
-  <xacro:property name="wheel_separation" value="0.56"/>
-  <xacro:property name="rear_wheel_offset" value="0.05"/>
-  <xacro:property name="base_length" value="0.6"/>
-  <xacro:property name="base_width" value="0.5"/>
+  <xacro:property name="wheel_width" value="0.07"/>
+  <xacro:property name="wheel_separation" value="0.455"/>
+  <xacro:property name="rear_wheel_offset" value="0.085"/>
+  <xacro:property name="base_length" value="0.65"/>
+  <xacro:property name="base_width" value="0.38"/>
   <xacro:property name="base_height" value="0.15"/>
   <xacro:property name="ground_clearance" value="0.09"/>
   <xacro:property name="front_wheel_radius" value="0.045"/>
-  <xacro:property name="front_wheel_offset" value="0.05"/>
+  <xacro:property name="front_wheel_offset" value="0.08"/>
   <!-- mower blades (piatti di taglio) -->
   <xacro:property name="blade_radius" value="0.11"/>
